File: light-sensor-module.kicad_pcb (KiCad board)
At the start: 2 copper layers, 36.8 x 29.2 mm, 18 parts, among them P1 MOLEX_01X06, P2 HEADER_01X06, P3 TERM_01X02, U1 STR05, U2 VEML6030, U3 BH1750

Commit message: Home computer branch
Parts:
- moved C7 3.81 mm to (133.3, 110.5), turned to 180 degrees
- moved C2 3.81 mm to (133.3, 114.3)
- moved R5 2.54 mm to (142.2, 114.3), turned to 180 degrees
- moved C1 2.54 mm to (142.2, 111.8), turned to 180 degrees
- moved R1 0.08 mm to (142.2, 101.6), turned to 180 degrees
- moved R2 0.08 mm to (142.2, 104.1), turned to 180 degrees
- moved R3 0.08 mm to (142.2, 106.7), turned to 180 degrees
- moved R4 0.08 mm to (142.2, 109.2), turned to 180 degrees
Routing:
- net DVI: track 18.7 -> 0.30 mm
- net SCL: track 5.76 -> 0.63 mm
