File: light-sensor-module.sch (KiCad schematic (older format))
At the start: 18 parts, among them P1 MOLEX_01X06, P2 HEADER_01X06, P3 TERM_01X02, U1 STR05, U2 VEML6030, U3 BH1750

Commit message: Home computer branch
Parts:
- L1: footprint ValveTeam_Library:WURTH_INDUCTOR -> valveteam-footprints:WURTH_INDUCTOR
- P3: footprint ValveTeam_Library:TE_TERM -> valveteam-footprints:TE_TERM
- U1: footprint ValveTeam_Library:STR05 -> valveteam-footprints:STR05
- U2: footprint ValveTeam_Library:VEML6030 -> valveteam-footprints:VEML6030
- U3: footprint ValveTeam_Library:WSOF6 -> valveteam-footprints:WSOF6
Changed lines of the file:
@@
 F 0 "U2" H 5650 3150 50  0000 C CNN
 F 1 "VEML6030" H 5650 2950 50  0000 C CNN
-F 2 "ValveTeam_Library:VEML6030" H 5650 3050 50  0001 C CNN
+F 2 "valveteam-footprints:VEML6030" H 5650 3050 50  0001 C CNN
 F 3 "" H 5650 3050 50  0000 C CNN
 	1    5650 3050
@@
 F 0 "U3" H 5650 5000 50  0000 C CNN
 F 1 "BH1750" H 5650 4800 50  0000 C CNN
-F 2 "ValveTeam_Library:WSOF6" H 5650 4900 50  0001 C CNN
+F 2 "valveteam-footprints:WSOF6" H 5650 4900 50  0001 C CNN
 F 3 "" H 5650 4900 50  0000 C CNN
 	1    5650 4900
@@
 F 0 "U1" H 3350 4154 50  0000 C CNN
 F 1 "STR05" H 3200 4550 50  0000 C CNN
-F 2 "ValveTeam_Library:STR05" H 3200 4350 50  0001 C CNN
+F 2 "valveteam-footprints:STR05" H 3200 4350 50  0001 C CNN
 F 3 "" H 3200 4350 50  0000 C CNN
 	1    3200 4350
@@
 F 0 "L1" V 2150 4300 50  0000 C CNN
 F 1 "3.3uH" V 2300 4300 50  0000 C CNN
-F 2 "ValveTeam_Library:WURTH_INDUCTOR" H 2200 4300 50  0001 C CNN
+F 2 "valveteam-footprints:WURTH_INDUCTOR" H 2200 4300 50  0001 C CNN
 F 3 "" H 2200 4300 50  0000 C CNN
 	1    2200 4300
@@
 F 0 "P3" H 1050 2950 50  0000 C CNN
 F 1 "TERM_01X02" V 1150 2800 50  0000 C CNN
-F 2 "ValveTeam_Library:TE_TERM" H 1050 2800 50  0001 C CNN
+F 2 "valveteam-footprints:TE_TERM" H 1050 2800 50  0001 C CNN
 F 3 "" H 1050 2800 50  0000 C CNN
 	1    1050 2800
