File: light-sensor-module.sch (KiCad schematic (older format))
At the start: 18 parts, among them P1 MOLEX_01X06, P2 HEADER_01X06, P3 TERM_01X02, U1 STR05, U2 VEML6030, U3 BH1750

Commit message: Complete PCB design
Parts:
- added D1, D2, D3, D4: LED, LEDs:LED_0805_HandSoldering, symbol LED
- added R6, R7, R8, R9: 470R, Resistors_SMD:R_0805_HandSoldering, symbol R
Connections:
- net DVI: now also R9.2
- net GNDREF: now also R6.2, R7.2
- net INT: now also R8.2
- net VCC+3: now also D2.2 (A), D3.2 (A), D4.2 (A)
- net VIN+12: now also D1.2 (A)
- new net: D1.1 (K), R6.1
- new net: D2.1 (K), R7.1
- new net: D3.1 (K), R8.1
- new net: D4.1 (K), R9.1
Other:
- moved on the sheet: C7, P1, P2, R4, R5
